File: Handy_sense_v_1.0.1.brd (EAGLE design)
At the start: 85 x 130.1 mm, 105 parts, among them K1 JS-M1-9V-4, K2 JS-M1-9V-4, K3 JS-M1-9V-4, K4 JS-M1-9V-4, Q1 600mA/40V, Q2 600mA/40V, Q3 600mA/40V, Q4 600mA/40V, Q5 600mA/40V, Q6 600mA/40V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

Commit message: ๊Update
Parts:
- removed C11, C9: 0.1uF, SparkFun-Capacitors:0805
- removed CONNECTOR1, CONNECTOR2, CONNECTOR3: (no value), con-lstb:MA03-1
- removed X1: (no value), con-wago-508:W237-4P
- added IO11_SW: TACTILE-SWITCH-PTH, GeekAmmo:TAC-SWITCH-PTH
- added R27: 10k, adafruit:R0805
- added X3, X9: (no value), con-wago-508:W237-132
- R12: value 10k -> 4.7k
- R25, R26, R5: value 1k -> 10k
- moved R3 8.95 mm to (71.8, 94.0)
- moved IO2_SW 4.04 mm to (66.4, 81.2), turned to 180 degrees
- moved R16 3.74 mm to (71.6, 89.3)
- moved R1 0.13 mm to (64.7, 89.5)
- renumbered 3.3V to LEDR1, 5V to LEDR2, DATA to LEDG1, WIFI to LEDB1
Connections:
- removed net VANALOG: CONNECTOR3.2, X11.1, X4.1, X5.1
- removed net VI2C_1: CONNECTOR2.2, X7.1
- removed net VI2C_2: CONNECTOR1.2, X10.1
- net 3.3V: now also IO11_SW.3, IO2_SW.3, X11.1, X4.1, X5.1; no longer C11.1, CONNECTOR1.1, CONNECTOR2.1, CONNECTOR3.1, R16.2
- net GND: now also R16.1, R27.1, X3.2; no longer C11.2, C9.2, IO2_SW.1, X1.2
- net GND2: now also X9.2; no longer X1.4
- net IO0: no longer C9.1
- net IO11: now also IO11_SW.1, R27.2
- net IO2: now also IO2_SW.1, R16.2; no longer IO2_SW.3, R16.1
- net N$28: now also X3.1; no longer X1.1
- net N$35: now also X9.1; no longer X1.3
- net VIN: now also X10.1, X7.1; no longer CONNECTOR1.3, CONNECTOR2.3, CONNECTOR3.3
Routing:
- net IO11: track 0.00 -> 58.8 mm, vias 0 -> 5
- net VANALOG: track 54.8 -> 0.00 mm
- net 3.3V: track 270.4 -> 310.7 mm, vias 13 -> 8
- net N$3: track 43.7 -> 29.8 mm, vias 4 -> 2
- net IO2: track 42.2 -> 55.6 mm
- net GND: track 635.5 -> 624.5 mm
- net VI2C_1: track 9.61 -> 0.00 mm
- net VI2C_2: track 9.21 -> 0.00 mm
- net VIN: track 283.8 -> 288.6 mm
- net IO32: track 70.5 -> 67.8 mm
- net MISO: track 108.6 -> 106.9 mm
- net RX2: track 115.6 -> 114.0 mm
- net TX2: track 101.7 -> 100.3 mm
- net SCL: track 152.5 -> 151.4 mm
- net IO4: track 105.9 -> 104.8 mm
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Other:
- board text added: "4.7k"
- board text added: "CLK"
- board text added: "CS/SS"
- board text added: "Handy Sense board"
- board text added: "MISO"
- board text added: "MOSI"
- board text added: "RX2"
- board text added: "TX2"
- board text removed: "5V"
- board text removed: "CLK/IO18"
- board text removed: "CS/SS/IO5"
- board text removed: "HandySense board"
- board text removed: "MISO/IO19"
- board text removed: "MOSI/IO23"
- board text removed: "RX2/IO16"
- board text removed: "TX2/IO17"
