File: Handy_sense_v_1.0.1.brd (EAGLE design)
At the start: 85 x 130.1 mm, 105 parts, among them K1 JS-M1-9V-4, K2 JS-M1-9V-4, K3 JS-M1-9V-4, K4 JS-M1-9V-4, Q1 600mA/40V, Q2 600mA/40V, Q3 600mA/40V, Q4 600mA/40V, Q5 600mA/40V, Q6 600mA/40V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

Commit message: Update
Parts:
- removed C11, C9: 0.1uF, SparkFun-Capacitors:0805
- R12: value 10k -> 4.7k
Connections:
- net 3.3V: no longer C11.1, X10.1, X7.1
- net GND: no longer C11.2, C9.2
- net IO0: no longer C9.1
- net VIN: now also X10.1, X7.1
Routing:
- net VIN: track 257.7 -> 288.6 mm, vias 5 -> 6
- net 3.3V: track 328.0 -> 310.7 mm, vias 9 -> 8
- net GND: track 630.7 -> 624.5 mm
- net IO0: track 64.6 -> 62.6 mm
Other:
- board text added: "4.7k"
