File: Handy_sense_v_1.0.1.sch (EAGLE design)
At the start: 105 parts, among them K1 JS-M1-9V-4, K2 JS-M1-9V-4, K3 JS-M1-9V-4, K4 JS-M1-9V-4, Q1 600mA/40V, Q2 600mA/40V, Q3 600mA/40V, Q4 600mA/40V, Q5 600mA/40V, Q6 600mA/40V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

Commit message: ๊Update
Parts:
- removed C11, C9: 0.1uF, SparkFun-Capacitors:CAP0805
- removed CONNECTOR1, CONNECTOR2, CONNECTOR3: (no value), con-lstb:MA03-1
- removed X1: (no value), con-wago-508:W237-04P
- added IO11_SW: TACTILE-SWITCH-PTH, GeekAmmo:TACTILE-SWITCH-PTH
- added R27: 10k, adafruit:R-US_R0805
- added X3, X9: (no value), con-wago-508:W237-02P
- R12: value 10k -> 4.7k
- R25, R26, R5: value 1k -> 10k
- renumbered 3.3V to LEDR1, 5V to LEDR2, DATA to LEDG1, WIFI to LEDB1
Connections:
- removed net VANALOG: CONNECTOR3.2, X11-1.KL, X4-1.KL, X5-1.KL
- removed net VI2C_1: CONNECTOR2.2, X7-1.KL
- removed net VI2C_2: CONNECTOR1.2, X10-1.KL
- net 3.3V: now also IO11_SW.3, IO2_SW.3, X11-1.KL, X4-1.KL, X5-1.KL; no longer C11.1, CONNECTOR1.1, CONNECTOR2.1, CONNECTOR3.1, R16.2
- net GND: now also R16.1, R27.1, X3-2.KL; no longer C11.2, C9.2, IO2_SW.1, X1-2.KL
- net GND2: now also X9-2.KL; no longer X1-4.KL
- net IO0: no longer C9.1
- net IO11: now also IO11_SW.1, R27.2
- net IO2: now also IO2_SW.1, R16.2; no longer IO2_SW.3, R16.1
- net N$28: now also X3-1.KL; no longer X1-1.KL
- net N$35: now also X9-1.KL; no longer X1-3.KL
- net VIN: now also X10-1.KL, X7-1.KL; no longer CONNECTOR1.3, CONNECTOR2.3, CONNECTOR3.3
Other:
- moved on the sheet: IO2_SW, R16
