File: Handy_sense_v_1.0.1.sch (EAGLE design)
At the start: 105 parts, among them K1 JS-M1-9V-4, K2 JS-M1-9V-4, K3 JS-M1-9V-4, K4 JS-M1-9V-4, Q1 600mA/40V, Q2 600mA/40V, Q3 600mA/40V, Q4 600mA/40V, Q5 600mA/40V, Q6 600mA/40V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

Commit message: Update
Parts:
- removed C11, C9: 0.1uF, SparkFun-Capacitors:CAP0805
- R12: value 10k -> 4.7k
Connections:
- net 3.3V: no longer C11.1, X10-1.KL, X7-1.KL
- net GND: no longer C11.2, C9.2
- net IO0: no longer C9.1
- net VIN: now also X10-1.KL, X7-1.KL
