File: Handy_sense_v_1.0.2.sch (EAGLE design)
At the start: 103 parts, among them K1 JS-M1-9V-4, K2 JS-M1-9V-4, K3 JS-M1-9V-4, K4 JS-M1-9V-4, Q1 600mA/40V, Q2 600mA/40V, Q3 600mA/40V, Q4 600mA/40V, Q5 600mA/40V, Q6 600mA/40V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

Commit message: Update version
- change tvs
- add 3.3 V and 5V
- change micro use
Parts:
- removed C12, C7: 10uF, SparkFun-Capacitors:10UF-16V-10%(TANT)
- removed CONNECTOR: (no value), con-lstb:MA03-1
- removed IO11_SW, IO2_SW: TACTILE-SWITCH-PTH, GeekAmmo:TACTILE-SWITCH-PTH
- removed J28CA2, J28CA5: (no value), DIOM505270X240:SMBJ28CA
- removed R27: 10k, adafruit:R-US_R0805
- removed USB: MICRO_USB_B_HIROSE_ZX62-B-5PA(11), connector:MICRO_USB_B_HIROSE_ZX62-B-5PA(11)
- added IO35_SW: TACTILE-SWITCH-PTH, GeekAmmo:TACTILE-SWITCH-PTH
- added JMP1, JMP2, JMP3, JMP4: 0R-JUMPB, jump-0r-smd:0R-JUMPB
- added MICRO_UDB: 629105136821, Wurth_Input-Output_Connectors_rev15d:629105136821
- R25, R26: value 10k -> 1k
- R3: value 22.1k -> 10k
- R8, R9: value 10k -> 4.7k
- renumbered LEDB1 to WIFI, LEDG1 to DATA, LEDR1 to 3.3V, LEDR2 to 5V
Connections:
- new net VA0: JMP2-0R.2, X4-1.KL
- new net VA3: JMP1-0R.2, X5-1.KL
- new net VA6: JMP3-0R.2, X11-1.KL
- net 3.3V: now also JMP1-0R.3, JMP2-0R.3, JMP3-0R.3, JMP4-0R.3, R16.2; no longer CONNECTOR.1, IDC10-1.KL, IO11_SW.3, IO2_SW.3, X11-1.KL, X4-1.KL, X5-1.KL
- net 5V: now also MICRO_UDB.+5V; no longer USB.+5V
- net GND: now also IO35_SW.1, MICRO_UDB.GND, MICRO_UDB.GND1, MICRO_UDB.GND2, MICRO_UDB.GND3, MICRO_UDB.GND4, MICRO_UDB.ID; no longer C7.-, J28CA2.J1, R16.1, R27.1, USB.GND
- net GND2: no longer C12.-, J28CA5.J1
- net IO11: no longer IO11_SW.1, R27.2
- net IO2: no longer IO2_SW.1, R16.2
- net IO35: now also IO35_SW.3, R16.1
- net K1CM: now also X2-2.KL; no longer X2-1.KL
- net K1NC: now also X2-3.KL; no longer X2-2.KL
- net K1NO: now also X2-1.KL; no longer X2-3.KL
- net K2CM: now also X12-2.KL; no longer X12-1.KL
- net K2NC: now also X12-3.KL; no longer X12-2.KL
- net K2NO: now also X12-1.KL; no longer X12-3.KL
- net K3CM: now also X6-2.KL; no longer X6-1.KL
- net K3NC: now also X6-3.KL; no longer X6-2.KL
- net K3NO: now also X6-1.KL; no longer X6-3.KL
- net K4CM: now also X8-2.KL; no longer X8-1.KL
- net K4NC: now also X8-3.KL; no longer X8-2.KL
- net K4NO: now also X8-1.KL; no longer X8-3.KL
- net N$34: no longer J28CA2.J2
- net N$37: no longer J28CA5.J2
- net RTCVCC: now also JMP4-0R.2; no longer CONNECTOR.2
- net USB_DN: now also MICRO_UDB.D-; no longer USB.D-
- net USB_DP: now also MICRO_UDB.D+; no longer USB.D+
- net VIN: now also IDC10-1.KL, JMP1-0R.1, JMP2-0R.1, JMP3-0R.1, JMP4-0R.1; no longer C7.+, CONNECTOR.3
- net VIN2: no longer C12.+
Other:
- moved on the sheet: D2, D3, IDC10-1, IDC10-10, IDC10-2, IDC10-3, IDC10-4, IDC10-5, IDC10-6, IDC10-7, IDC10-8, IDC10-9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
